File: Weather Shield.brd (EAGLE design)
At the start: 83.8 x 55.9 mm, 38 parts, among them Q1 BSS138, Q2 BSS138, U1 DS3231SN, U4 MPL3115A2LGA8, U5 HTU21D

Commit message: routing...
Parts:
- moved U1 8.13 mm to (36.8, 33.0)
Changed lines of the file:
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@@
 </element>
 <element name="LOGO1" library="SparkFun-Aesthetics" package="OSHW-LOGO-M" value="OSHW-LOGOM" x="58.42" y="44.45"/>
-<element name="U1" library="FSE_Weather_Shield" package="SOIC127P1032X265-16N" value="DS3231SN" x="43.18" y="38.1" rot="R90">
-<attribute name="SUPPLIER" value="Maxim" x="43.18" y="38.1" size="1.778" layer="27" rot="R90" display="off"/>
-<attribute name="PACKAGE" value="SOIC-16" x="43.18" y="38.1" size="1.778" layer="27" rot="R90" display="off"/>
-<attribute name="MPN" value="DS3231SN#" x="43.18" y="38.1" size="1.778" layer="27" rot="R90" display="off"/>
-<attribute name="OC_FARNELL" value="1593292" x="43.18" y="38.1" size="1.778" layer="27" rot="R90" display="off"/>
-<attribute name="OC_NEWARK" value="68K3406" x="43.18" y="38.1" size="1.778" layer="27" rot="R90" display="off"/>
+<element name="U1" library="FSE_Weather_Shield" package="SOIC127P1032X265-16N" value="DS3231SN" x="36.83" y="33.02" rot="R90">
+<attribute name="SUPPLIER" value="Maxim" x="36.83" y="33.02" size="1.778" layer="27" rot="R90" display="off"/>
+<attribute name="PACKAGE" value="SOIC-16" x="36.83" y="33.02" size="1.778" layer="27" rot="R90" display="off"/>
+<attribute name="MPN" value="DS3231SN#" x="36.83" y="33.02" size="1.778" layer="27" rot="R90" display="off"/>
+<attribute name="OC_FARNELL" value="1593292" x="36.83" y="33.02" size="1.778" layer="27" rot="R90" display="off"/>
+<attribute name="OC_NEWARK" value="68K3406" x="36.83" y="33.02" size="1.778" layer="27" rot="R90" display="off"/>
 </element>
 <element name="C1" library="SparkFun" package="0603-CAP" value="0.1uF" x="54.61" y="33.02" rot="R180"/>
@@
 <contactref element="PCB1" pad="39"/>
 <wire x1="53.76" y1="33.02" x2="64.77" y2="35.56" width="0" layer="19" extent="1-1"/>
-<wire x1="47.625" y1="33.401" x2="53.76" y2="33.02" width="0" layer="19" extent="1-1"/>
-<wire x1="46.355" y1="33.401" x2="47.625" y2="33.401" width="0" layer="19" extent="1-1"/>
-<wire x1="45.085" y1="33.401" x2="46.355" y2="33.401" width="0" layer="19" extent="1-1"/>
-<wire x1="43.815" y1="33.401" x2="45.085" y2="33.401" width="0" layer="19" extent="1-1"/>
-<wire x1="47.625" y1="42.799" x2="47.625" y2="33.401" width="0" layer="19" extent="1-1"/>
-<wire x1="46.355" y1="42.799" x2="47.625" y2="42.799" width="0" layer="19" extent="1-1"/>
-<wire x1="45.085" y1="42.799" x2="46.355" y2="42.799" width="0" layer="19" extent="1-1"/>
-<wire x1="43.815" y1="42.799" x2="45.085" y2="42.799" width="0" layer="19" extent="1-1"/>
-<wire x1="42.545" y1="42.799" x2="43.815" y2="42.799" width="0" layer="19" extent="1-1"/>
-<wire x1="20.32" y1="45.3" x2="42.545" y2="42.799" width="0" layer="19" extent="1-1"/>
+<wire x1="41.275" y1="28.321" x2="53.76" y2="33.02" width="0" layer="19" extent="1-1"/>
+<wire x1="40.005" y1="28.321" x2="41.275" y2="28.321" width="0" layer="19" extent="1-1"/>
+<wire x1="38.735" y1="28.321" x2="40.005" y2="28.321" width="0" layer="19" extent="1-1"/>
+<wire x1="37.465" y1="28.321" x2="38.735" y2="28.321" width="0" layer="19" extent="1-1"/>
+<wire x1="41.275" y1="37.719" x2="41.275" y2="28.321" width="0" layer="19" extent="1-1"/>
+<wire x1="40.005" y1="37.719" x2="41.275" y2="37.719" width="0" layer="19" extent="1-1"/>
+<wire x1="38.735" y1="37.719" x2="40.005" y2="37.719" width="0" layer="19" extent="1-1"/>
+<wire x1="37.465" y1="37.719" x2="38.735" y2="37.719" width="0" layer="19" extent="1-1"/>
+<wire x1="36.195" y1="37.719" x2="37.465" y2="37.719" width="0" layer="19" extent="1-1"/>
+<wire x1="20.32" y1="45.3" x2="36.195" y2="37.719" width="0" layer="19" extent="1-1"/>
 <wire x1="20.32" y1="49.11" x2="20.32" y2="45.3" width="0" layer="19" extent="1-1"/>
 <wire x1="17.78" y1="40.76" x2="20.32" y2="45.3" width="0" layer="19" extent="1-1"/>
@@
 <contactref element="U1" pad="2"/>
 <contactref element="C1" pad="1"/>
-<wire x1="40.005" y1="33.401" x2="55.46" y2="33.02" width="0" layer="19" extent="1-1"/>
+<wire x1="33.655" y1="28.321" x2="55.46" y2="33.02" width="0" layer="19" extent="1-1"/>
 </signal>
 <signal name="N$6">
@@
 <contactref element="U1" pad="14"/>
 <wire x1="64.77" y1="28.955" x2="64.77" y2="42.165" width="0" layer="19" extent="1-1"/>
-<wire x1="41.275" y1="42.799" x2="64.77" y2="28.955" width="0" layer="19" extent="1-1"/>
+<wire x1="34.925" y1="37.719" x2="64.77" y2="28.955" width="0" layer="19" extent="1-1"/>
 </signal>
 <signal name="5V0">

Commit message: initial project version
Parts:
- added D2: Blue, SparkFun:LED-0603
- added R7: 1K, rcl:R0603
- JP9-DNP1, JP9-DNP2: value RJ11-RAIN -> (none)
- moved LOGO1 63.8 mm to (3.81, 11.4)
- moved JP9-DNP1 18.2 mm to (45.7, 5.08), turned to 0 degrees
- moved U1 9.16 mm to (44.5, 38.1)
- moved G1 5.24 mm to (63.5, 40.6)
Connections:
- new net N$10: D2.A, R7.2
- new net STAT3: R7.1
- net GND: now also D2.C
- net SCL: now also U1.16
- net SDA: now also U1.15
Other:
- board size 83.8 x 55.9 mm -> 30.5 x 35.6 mm

Commit message: initial project version
Parts:
- moved JP9-DNP2 1.80 mm to (99.1, 27.9)
Changed lines of the file:
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@@
 <element name="PCB1" library="FSE_Weather_Shield" package="RASPBERRY_PI_BPLUS_DIM" value="RASPBERRY_PI_B+/PI2_DIM" x="0" y="0"/>
 <element name="JP9-DNP1" library="SparkFun" package="RJ11-6" value="" x="45.72" y="5.08"/>
-<element name="JP9-DNP2" library="SparkFun" package="RJ11-6" value="" x="97.79" y="26.67" rot="R90"/>
+<element name="JP9-DNP2" library="SparkFun" package="RJ11-6" value="" x="99.06" y="27.94" rot="R90"/>
 <element name="R7" library="rcl" package="R0603" value="1K" x="-6.35" y="-27.94"/>
 <element name="D2" library="SparkFun" package="LED-0603" value="Blue" x="-6.35" y="-31.75"/>
