File: WeatherShield.brd (EAGLE design)
At the start: 90.3 x 67.3 mm, 78 parts, among them Q1 BSS138, Q2 BSS138, U1 DS3231SN, U2 LT3652, U4 MPL3115A2LGA8, U5 HTU21D

Commit message: WeatherShield_v1
Parts:
- removed U$2: DEAN_CONNECTOR, FSE_Weather_Shield:DEAN_CONNECTOR
- removed U$3: V_BATT, FSE_Weather_Shield:DEAN_CONNECTOR
- added U$1, U$6: XT-60, FSEWeatherShield:XT-60
- moved C8 15.3 mm to (52.1, 41.7), turned to 0 degrees
- moved G1 4.07 mm to (54.1, 50.8)
- moved C1 3.16 mm to (52.2, 40.7), turned to 0 degrees
Connections:
- removed net +5V: C16.1, C17.1, C18.+, C19.1, L1.2, R19.2, U$4.5
- removed net VCC: C1.1, JP9-DNP1.2, JP9-DNP2.2, PCB1.1, PCB1.17, U1.2
- net 3.3V: now also C1.1, JP9-DNP1.2, JP9-DNP2.2, PCB1.1, PCB1.17, U1.2
- net 5V: now also C16.1, C17.1, C18.+, C19.1, L1.2, R19.2, U$4.5
- net GND: now also U$1.NEG, U$6.NEG; no longer U$2.2, U$3.2
- net VIN: now also U$1.POS; no longer U$2.1
- net V_BATT: now also U$6.POS; no longer U$3.1
Routing:
- net VCC: track 98.2 -> 0.00 mm, vias 1 -> 0
- net +5V: track 50.8 -> 2.90 mm, vias 2 -> 0
- net N$6: track 31.0 -> 0.00 mm, vias 1 -> 0
- net V_BATT: track 70.9 -> 58.6 mm
- net VIN: track 26.1 -> 23.4 mm
Other:
- outline, holes or cut-outs redrawn
