File: AirBoard_Shield/WeatherShield_Air.brd (EAGLE design)
At the start: 33 x 26.7 mm, 8 parts, among them U4 MPL3115A2LGA8, U5 HTU21D

Commit message: WeatherShield v1
Parts:
- R25: value 1K -> 280
- moved LOGO1 23.5 mm to (28.8, 4.06)
- moved D12 21.4 mm to (21.7, 24.0), turned to 180 degrees
- moved R25 21.0 mm to (23.2, 23.2), turned to 90 degrees
- moved C6 10.1 mm to (13.8, 15.7), turned to 0 degrees
- moved JP9-DNP2 4.06 mm to (33.9, 7.98)
- moved U4 3.33 mm to (13.6, 19.9), turned to 90 degrees
- moved C5 2.79 mm to (14.0, 5.21), turned to 0 degrees
- moved U5 1.89 mm to (13.1, 9.53), turned to 90 degrees
Connections:
- removed net STAT1: R25.1
- net 5V: now also R25.1
Routing:
- net 3.3V: track 0.00 -> 12.5 mm
- net SDA: track 0.00 -> 11.2 mm
- net 5V: track 0.00 -> 5.83 mm
- net N$5: track 0.00 -> 3.00 mm
- net N$28: track 0.00 -> 1.80 mm
Changed lines of the file:
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@@
 <board>
 <plain>
-<text x="11.557" y="0.381" size="1.016" layer="21" ratio="15">FSE Weather Shield V1</text>
+<text x="8.128" y="1.397" size="1.016" layer="21" ratio="15">FSE Weather Shield V1</text>
 <text x="22.86" y="-24.13" size="1.778" layer="27" font="vector" ratio="15">N. Seidle</text>
-<text x="22.606" y="24.892" size="1.27" layer="21" ratio="15" rot="R180">Pressure</text>
-<text x="2.667" y="14.732" size="1.27" layer="21" ratio="15">Humidity</text>
+<text x="8.636" y="12.573" size="1.27" layer="21" ratio="15" rot="R270">Pressure</text>
+<text x="7.747" y="12.192" size="1.27" layer="21" ratio="15" rot="R90">Humidity</text>
 <wire x1="33.274" y1="22.733" x2="33.274" y2="3.683" width="0" layer="20"/>
 <wire x1="0.254" y1="22.733" x2="0.254" y2="3.683" width="0" layer="20"/>
@@
 </autorouter>
 <elements>
-<element name="U4" library="SparkFun-Sensors" package="LGA8" value="MPL3115A2LGA8" x="16.764" y="18.923"/>
-<element name="C6" library="rcl" package="C0603" value="0.1uF" x="17.78" y="6.477" smashed="yes" rot="R270">
-<attribute name="NAME" x="18.542" y="7.366" size="0.8128" layer="25" font="vector" rot="R270"/>
-<attribute name="VALUE" x="16.637" y="7.493" size="0.8128" layer="27" font="vector" rot="R270"/>
+<element name="U4" library="SparkFun-Sensors" package="LGA8" value="MPL3115A2LGA8" x="13.589" y="19.939" rot="R90"/>
+<element name="C6" library="rcl" package="C0603" value="0.1uF" x="13.843" y="15.748" smashed="yes">
+<attribute name="NAME" x="12.954" y="16.51" size="0.8128" layer="25" font="vector"/>
+<attribute name="VALUE" x="12.827" y="14.605" size="0.8128" layer="27" font="vector"/>
 </element>
-<element name="C5" library="rcl" package="C0603" value="0.1uF" x="13.97" y="8.001" smashed="yes" rot="R180">
-<attribute name="NAME" x="14.859" y="7.239" size="0.8128" layer="25" font="vector" rot="R180"/>
-<attribute name="VALUE" x="14.986" y="9.144" size="0.8128" layer="27" font="vector" rot="R180"/>
+<element name="C5" library="rcl" package="C0603" value="0.1uF" x="13.97" y="5.207" smashed="yes">
+<attribute name="NAME" x="13.081" y="5.969" size="0.8128" layer="25" font="vector"/>
+<attribute name="VALUE" x="12.954" y="4.064" size="0.8128" layer="27" font="vector"/>
 </element>
-<element name="U5" library="SparkFun-Sensors" package="HTU21D" value="HTU21D" x="14.478" y="10.795" smashed="yes">
-<attribute name="NAME" x="13.403" y="12.57" size="0.8128" layer="25"/>
-<attribute name="VALUE" x="13.153" y="8.595" size="0.8128" layer="27"/>
+<element name="U5" library="SparkFun-Sensors" package="HTU21D" value="HTU21D" x="13.081" y="9.525" smashed="yes" rot="R90">
+<attribute name="NAME" x="11.306" y="8.45" size="0.8128" layer="25" rot="R90"/>
+<attribute name="VALUE" x="15.281" y="8.2" size="0.8128" layer="27" rot="R90"/>
 </element>
-<element name="LOGO1" library="SparkFun-Aesthetics" package="OSHW-LOGO-M" value="OSHW-LOGOM" x="5.334" y="3.683" rot="R90"/>
-<element name="JP9-DNP2" library="FSEWeatherShield" package="RJ11-STECKER" value="RJ11-BUCHSE" x="33.9344" y="3.9116" rot="R90"/>
-<element name="R25" library="rcl" package="R0603" value="1K" x="17.78" y="2.921" rot="R270"/>
-<element name="D12" library="SparkFun" package="LED-0603" value="AirBoard status led" x="16.002" y="3.429"/>
+<element name="LOGO1" library="SparkFun-Aesthetics" package="OSHW-LOGO-M" value="OSHW-LOGOM" x="28.829" y="4.064" rot="R90"/>
+<element name="JP9-DNP2" library="FSEWeatherShield" package="RJ11-STECKER" value="RJ11-BUCHSE" x="33.9344" y="7.9756" rot="R90"/>
+<element name="R25" library="rcl" package="R0603" value="280" x="23.241" y="23.241" rot="R90"/>
+<element name="D12" library="SparkFun" package="LED-0603" value="AirBoard status led" x="21.717" y="24.003" rot="R180"/>
 </elements>
 <signals>
@@
 <contactref element="U5" pad="GND"/>
 <contactref element="C5" pad="2"/>
-<polygon width="0.4064" layer="1">
+<polygon width="0.4064" layer="1" isolate="0.3048">
 <vertex x="0.254" y="27.813"/>
 <vertex x="33.528" y="27.559"/>
@@
 <contactref element="JP9-DNP2" pad="5"/>
 <contactref element="JP9-DNP2" pad="6"/>
-<wire x1="23.0944" y1="8.4816" x2="25.6344" y2="7.4616" width="0" layer="19" extent="1-1"/>
-<wire x1="17.78" y1="5.627" x2="23.0944" y2="8.4816" width="0" layer="19" extent="1-1"/>
-<wire x1="16.002" y1="4.179" x2="17.78" y2="5.627" width="0" layer="19" extent="1-1"/>
-<wire x1="13.12" y1="8.001" x2="16.002" y2="4.179" width="0" layer="19" extent="1-1"/>
-<wire x1="14.478" y1="10.795" x2="13.12" y2="8.001" width="0" layer="19" extent="1-1"/>
-<wire x1="15.978" y1="10.795" x2="14.478" y2="10.795" width="0" layer="19" extent="1-1"/>
-<wire x1="15.564" y1="18.298" x2="15.978" y2="10.795" width="0" layer="19" extent="1-1"/>
 </signal>
 <signal name="3.3V">
@@
 <contactref element="C5" pad="1"/>
 <contactref element="JP9-DNP2" pad="2"/>
-<wire x1="14.82" y1="8.001" x2="25.6344" y2="11.5416" width="0" layer="19" extent="1-1"/>
-<wire x1="12.978" y1="10.795" x2="14.82" y2="8.001" width="0" layer="19" extent="1-1"/>
-<wire x1="15.564" y1="17.048" x2="12.978" y2="10.795" width="0" layer="19" extent="1-1"/>
-<wire x1="15.564" y1="20.798" x2="15.564" y2="17.048" width="0" layer="19" extent="1-1"/>
+<wire x1="25.6344" y1="15.6056" x2="16.7794" y2="15.6056" width="0.4064" layer="1"/>
+<wire x1="16.7794" y1="15.6056" x2="15.494" y2="16.891" width="0.4064" layer="1"/>
+<wire x1="15.494" y1="16.891" x2="15.494" y2="18.709" width="0.4064" layer="1"/>
+<wire x1="15.494" y1="18.709" x2="15.464" y2="18.739" width="0.4064" layer="1"/>
+<wire x1="11.714" y1="18.739" x2="15.464" y2="18.739" width="0" layer="19" extent="1-1"/>
+<wire x1="13.081" y1="8.025" x2="16.7794" y2="15.6056" width="0" layer="19" extent="1-1"/>
+<wire x1="13.12" y1="5.207" x2="13.081" y2="8.025" width="0" layer="19" extent="1-1"/>
 </signal>
 <signal name="SCL">
@@
 <contactref element="U5" pad="SCK"/>
 <contactref element="JP9-DNP2" pad="4"/>
-<wire x1="12.978" y1="9.795" x2="25.6344" y2="9.5016" width="0" layer="19" extent="1-1"/>
-<wire x1="17.964" y1="20.798" x2="12.978" y2="9.795" width="0" layer="19" extent="1-1"/>
+<wire x1="14.081" y1="8.025" x2="25.6344" y2="13.5656" width="0" layer="19" extent="1-1"/>
+<wire x1="11.714" y1="21.139" x2="14.081" y2="8.025" width="0" layer="19" extent="1-1"/>
 </signal>
 <signal name="SDA">
@@
 <contactref element="U5" pad="DATA"/>
 <contactref element="JP9-DNP2" pad="3"/>
-<wire x1="15.978" y1="9.795" x2="23.0944" y2="10.5216" width="0" layer="19" extent="1-1"/>
-<wire x1="17.964" y1="19.548" x2="15.978" y2="9.795" width="0" layer="19" extent="1-1"/>
+<wire x1="23.0944" y1="14.5856" x2="16.3636" y2="14.5856" width="0.4064" layer="1"/>
+<wire x1="16.3636" y1="14.5856" x2="14.097" y2="12.319" width="0.4064" layer="1"/>
+<wire x1="14.097" y1="12.319" x2="14.097" y2="11.041" width="0.4064" layer="1"/>
+<wire x1="14.097" y1="11.041" x2="14.081" y2="11.025" width="0.4064" layer="1"/>
+<wire x1="16.3636" y1="14.5856" x2="12.964" y2="21.139" width="0" layer="19" extent="1-1"/>
 </signal>
 <signal name="INT-PRESSURE">
@@
 <contactref element="U4" pad="2"/>
 <contactref element="C6" pad="1"/>
-<wire x1="15.564" y1="19.548" x2="17.78" y2="7.327" width="0" layer="19" extent="1-1"/>
+<wire x1="12.993" y1="15.748" x2="12.993" y2="18.71" width="0.4064" layer="1"/>
+<wire x1="12.993" y1="18.71" x2="12.964" y2="18.739" width="0.4064" layer="1"/>
 </signal>
 <signal name="5V">
 <contactref element="JP9-DNP2" pad="1"/>
-</signal>
-<signal name="N$8">
-<via x="5.334" y="21.463" extent="1-16" drill="2.75" diameter="6.4516"/>
-</signal>
-<signal name="N$9">
-<via x="28.194" y="21.463" extent="1-16" drill="2.75" diameter="6.4516"/>
-</signal>
-<signal name="STAT1">
 <contactref element="R25" pad="1"/>
+<wire x1="23.241" y1="22.391" x2="23.241" y2="16.7722" width="0.4064" layer="1"/>
+<wire x1="23.241" y1="16.7722" x2="23.0944" y2="16.6256" width="0.4064" layer="1"/>
 </signal>
 <signal name="N$28">
 <contactref element="R25" pad="2"/>
 <contactref element="D12" pad="A"/>
-<wire x1="16.002" y1="2.679" x2="17.78" y2="2.071" width="0" layer="19" extent="1-1"/>
+<wire x1="21.717" y1="24.753" x2="22.579" y2="24.753" width="0.4064" layer="1"/>
+<wire x1="22.579" y1="24.753" x2="23.241" y2="24.091" width="0.4064" layer="1"/>
+</signal>
+<signal name="N$1">
+<via x="4.54" y="22.2" extent="1-16" drill="2.75" diameter="6.4516"/>
+</signal>
+<signal name="N$2">
+<via x="4.54" y="4.47" extent="1-16" drill="2.75" diameter="6.4516"/>
 </signal>
 </signals>

Commit message: WeatherShield_v1
Parts:
- moved C6 2.62 mm to (11.3, 16.4)
- moved R25 2.27 mm to (22.2, 21.2), turned to 180 degrees
- moved D12 1.90 mm to (20.6, 22.5), turned to 90 degrees
- moved C5 1.53 mm to (14.1, 6.73)
Routing:
- net SCL: track 0.00 -> 43.1 mm
- net 3.3V: track 12.5 -> 45.8 mm
- net SDA: track 11.2 -> 38.7 mm
- net GND: track 0.00 -> 12.7 mm, vias 0 -> 2
- net N$5: track 3.00 -> 4.27 mm
- net 5V: track 5.83 -> 4.59 mm
- net N$28: track 1.80 -> 1.29 mm
Changed lines of the file:
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@@
 <elements>
 <element name="U4" library="SparkFun-Sensors" package="LGA8" value="MPL3115A2LGA8" x="13.589" y="19.939" rot="R90"/>
-<element name="C6" library="rcl" package="C0603" value="0.1uF" x="13.843" y="15.748" smashed="yes">
-<attribute name="NAME" x="12.954" y="16.51" size="0.8128" layer="25" font="vector"/>
-<attribute name="VALUE" x="12.827" y="14.605" size="0.8128" layer="27" font="vector"/>
+<element name="C6" library="rcl" package="C0603" value="0.1uF" x="11.303" y="16.383" smashed="yes">
+<attribute name="NAME" x="10.414" y="17.145" size="0.8128" layer="25" font="vector"/>
+<attribute name="VALUE" x="10.287" y="15.24" size="0.8128" layer="27" font="vector"/>
 </element>
-<element name="C5" library="rcl" package="C0603" value="0.1uF" x="13.97" y="5.207" smashed="yes">
-<attribute name="NAME" x="13.081" y="5.969" size="0.8128" layer="25" font="vector"/>
-<attribute name="VALUE" x="12.954" y="4.064" size="0.8128" layer="27" font="vector"/>
+<element name="C5" library="rcl" package="C0603" value="0.1uF" x="14.097" y="6.731" smashed="yes">
+<attribute name="NAME" x="13.208" y="7.493" size="0.8128" layer="25" font="vector"/>
+<attribute name="VALUE" x="13.081" y="5.588" size="0.8128" layer="27" font="vector"/>
 </element>
 <element name="U5" library="SparkFun-Sensors" package="HTU21D" value="HTU21D" x="13.081" y="9.525" smashed="yes" rot="R90">
@@
 <element name="LOGO1" library="SparkFun-Aesthetics" package="OSHW-LOGO-M" value="OSHW-LOGOM" x="28.829" y="4.064" rot="R90"/>
 <element name="JP9-DNP2" library="FSEWeatherShield" package="RJ11-STECKER" value="RJ11-BUCHSE" x="33.9344" y="7.9756" rot="R90"/>
-<element name="R25" library="rcl" package="R0603" value="280" x="23.241" y="23.241" rot="R90"/>
-<element name="D12" library="SparkFun" package="LED-0603" value="AirBoard status led" x="21.717" y="24.003" rot="R180"/>
+<element name="R25" library="rcl" package="R0603" value="280" x="22.225" y="21.209" rot="R180"/>
+<element name="D12" library="SparkFun" package="LED-0603" value="AirBoard status led" x="20.574" y="22.479" rot="R90"/>
 </elements>
 <signals>
@@
 <contactref element="JP9-DNP2" pad="5"/>
 <contactref element="JP9-DNP2" pad="6"/>
+<wire x1="14.947" y1="6.731" x2="16.51" y2="6.731" width="0.4064" layer="1"/>
+<wire x1="16.51" y1="6.731" x2="19.05" y2="9.271" width="0.4064" layer="1"/>
+<via x="19.05" y="9.271" extent="1-16" drill="0.6"/>
+<wire x1="19.05" y1="9.271" x2="17.018" y2="11.303" width="0.4064" layer="16"/>
+<via x="17.018" y="11.303" extent="1-16" drill="0.6"/>
+<wire x1="17.018" y1="11.303" x2="15.24" y2="9.525" width="0.4064" layer="1"/>
+<wire x1="15.24" y1="9.525" x2="13.081" y2="9.525" width="0.4064" layer="1"/>
 </signal>
 <signal name="3.3V">
@@
 <contactref element="C5" pad="1"/>
 <contactref element="JP9-DNP2" pad="2"/>
-<wire x1="25.6344" y1="15.6056" x2="16.7794" y2="15.6056" width="0.4064" layer="1"/>
-<wire x1="16.7794" y1="15.6056" x2="15.494" y2="16.891" width="0.4064" layer="1"/>
-<wire x1="15.494" y1="16.891" x2="15.494" y2="18.709" width="0.4064" layer="1"/>
 <wire x1="15.494" y1="18.709" x2="15.464" y2="18.739" width="0.4064" layer="1"/>
-<wire x1="11.714" y1="18.739" x2="15.464" y2="18.739" width="0" layer="19" extent="1-1"/>
-<wire x1="13.081" y1="8.025" x2="16.7794" y2="15.6056" width="0" layer="19" extent="1-1"/>
-<wire x1="13.12" y1="5.207" x2="13.081" y2="8.025" width="0" layer="19" extent="1-1"/>
+<wire x1="13.247" y1="6.731" x2="13.081" y2="6.477" width="0.4064" layer="1"/>
+<wire x1="13.081" y1="6.477" x2="13.081" y2="8.025" width="0.4064" layer="1"/>
+<wire x1="11.714" y1="18.739" x2="9.214" y2="18.739" width="0.4064" layer="1"/>
+<wire x1="9.214" y1="18.739" x2="8.128" y2="17.653" width="0.4064" layer="1"/>
+<wire x1="8.128" y1="17.653" x2="8.128" y2="14.605" width="0.4064" layer="1"/>
+<wire x1="8.128" y1="14.605" x2="8.89" y2="13.843" width="0.4064" layer="1"/>
+<wire x1="8.89" y1="13.843" x2="9.144" y2="13.843" width="0.4064" layer="1"/>
+<wire x1="9.144" y1="13.843" x2="13.97" y2="13.843" width="0.4064" layer="1"/>
+<wire x1="13.97" y1="13.843" x2="15.621" y2="15.494" width="0.4064" layer="1"/>
+<wire x1="15.621" y1="15.494" x2="15.621" y2="18.582" width="0.4064" layer="1"/>
+<wire x1="15.621" y1="18.582" x2="15.464" y2="18.739" width="0.4064" layer="1"/>
+<wire x1="25.6344" y1="15.6056" x2="15.7326" y2="15.6056" width="0.4064" layer="1"/>
+<wire x1="15.7326" y1="15.6056" x2="15.621" y2="15.494" width="0.4064" layer="1"/>
+<wire x1="13.081" y1="8.025" x2="13.081" y2="5.461" width="0.4064" layer="1"/>
+<wire x1="13.081" y1="5.461" x2="12.827" y2="5.207" width="0.4064" layer="1"/>
+<wire x1="12.827" y1="5.207" x2="9.906" y2="5.207" width="0.4064" layer="1"/>
+<wire x1="9.906" y1="5.207" x2="8.89" y2="6.223" width="0.4064" layer="1"/>
+<wire x1="8.89" y1="6.223" x2="8.89" y2="13.589" width="0.4064" layer="1"/>
+<wire x1="8.89" y1="13.589" x2="9.144" y2="13.843" width="0.4064" layer="1"/>
 </signal>
 <signal name="SCL">
@@
 <contactref element="U5" pad="SCK"/>
 <contactref element="JP9-DNP2" pad="4"/>
-<wire x1="14.081" y1="8.025" x2="25.6344" y2="13.5656" width="0" layer="19" extent="1-1"/>
-<wire x1="11.714" y1="21.139" x2="14.081" y2="8.025" width="0" layer="19" extent="1-1"/>
+<wire x1="25.6344" y1="13.5656" x2="21.3126" y2="13.5656" width="0.4064" layer="1"/>
+<wire x1="21.3126" y1="13.5656" x2="15.748" y2="8.001" width="0.4064" layer="1"/>
+<wire x1="15.748" y1="8.001" x2="14.105" y2="8.001" width="0.4064" layer="1"/>
+<wire x1="14.105" y1="8.001" x2="14.081" y2="8.025" width="0.4064" layer="1"/>
+<wire x1="11.714" y1="21.139" x2="11.714" y2="22.89" width="0.4064" layer="1"/>
+<wire x1="11.714" y1="22.89" x2="12.7" y2="23.876" width="0.4064" layer="1"/>
+<wire x1="12.7" y1="23.876" x2="17.018" y2="23.876" width="0.4064" layer="1"/>
+<wire x1="17.018" y1="23.876" x2="18.034" y2="24.892" width="0.4064" layer="1"/>
+<wire x1="18.034" y1="24.892" x2="23.622" y2="24.892" width="0.4064" layer="1"/>
+<wire x1="25.6344" y1="13.5656" x2="26.7736" y2="13.5656" width="0.4064" layer="1"/>
+<wire x1="26.7736" y1="13.5656" x2="27.94" y2="14.732" width="0.4064" layer="1"/>
+<wire x1="27.94" y1="14.732" x2="27.94" y2="17.145" width="0.4064" layer="1"/>
+<wire x1="27.94" y1="17.145" x2="25.781" y2="19.304" width="0.4064" layer="1"/>
+<wire x1="25.781" y1="19.304" x2="25.781" y2="22.733" width="0.4064" layer="1"/>
+<wire x1="25.781" y1="22.733" x2="23.622" y2="24.892" width="0.4064" layer="1"/>
 </signal>
 <signal name="SDA">
@@
 <wire x1="14.097" y1="12.319" x2="14.097" y2="11.041" width="0.4064" layer="1"/>
 <wire x1="14.097" y1="11.041" x2="14.081" y2="11.025" width="0.4064" layer="1"/>
-<wire x1="16.3636" y1="14.5856" x2="12.964" y2="21.139" width="0" layer="19" extent="1-1"/>
+<wire x1="12.964" y1="21.139" x2="12.964" y2="22.235" width="0.4064" layer="1"/>
+<wire x1="12.964" y1="22.235" x2="13.589" y2="22.86" width="0.4064" layer="1"/>
+<wire x1="13.589" y1="22.86" x2="17.653" y2="22.86" width="0.4064" layer="1"/>
+<wire x1="17.653" y1="22.86" x2="18.669" y2="23.876" width="0.4064" layer="1"/>
+<wire x1="18.669" y1="23.876" x2="23.241" y2="23.876" width="0.4064" layer="1"/>
+<wire x1="23.241" y1="23.876" x2="24.13" y2="22.987" width="0.4064" layer="1"/>
+<wire x1="24.13" y1="22.987" x2="24.13" y2="18.161" width="0.4064" layer="1"/>
+<wire x1="24.13" y1="18.161" x2="25.146" y2="17.145" width="0.4064" layer="1"/>
+<wire x1="23.0944" y1="14.5856" x2="26.5236" y2="14.5856" width="0.4064" layer="1"/>
+<wire x1="26.5236" y1="14.5856" x2="27.051" y2="15.113" width="0.4064" layer="1"/>
+<wire x1="27.051" y1="15.113" x2="27.051" y2="16.764" width="0.4064" layer="1"/>
+<wire x1="27.051" y1="16.764" x2="26.67" y2="17.145" width="0.4064" layer="1"/>
+<wire x1="26.67" y1="17.145" x2="25.146" y2="17.145" width="0.4064" layer="1"/>
 </signal>
 <signal name="INT-PRESSURE">
@@
 <contactref element="U4" pad="2"/>
 <contactref element="C6" pad="1"/>
-<wire x1="12.993" y1="15.748" x2="12.993" y2="18.71" width="0.4064" layer="1"/>
 <wire x1="12.993" y1="18.71" x2="12.964" y2="18.739" width="0.4064" layer="1"/>
+<wire x1="12.993" y1="18.71" x2="12.993" y2="18.2" width="0.4064" layer="1"/>
+<wire x1="12.993" y1="18.2" x2="12.319" y2="17.526" width="0.4064" layer="1"/>
+<wire x1="12.319" y1="17.526" x2="10.922" y2="17.526" width="0.4064" layer="1"/>
+<wire x1="10.922" y1="17.526" x2="10.414" y2="17.018" width="0.4064" layer="1"/>
+<wire x1="10.414" y1="17.018" x2="10.414" y2="16.422" width="0.4064" layer="1"/>
+<wire x1="10.414" y1="16.422" x2="10.453" y2="16.383" width="0.4064" layer="1"/>
 </signal>
 <signal name="5V">
 <contactref element="JP9-DNP2" pad="1"/>
 <contactref element="R25" pad="1"/>
-<wire x1="23.241" y1="22.391" x2="23.241" y2="16.7722" width="0.4064" layer="1"/>
-<wire x1="23.241" y1="16.7722" x2="23.0944" y2="16.6256" width="0.4064" layer="1"/>
+<wire x1="23.0944" y1="16.6256" x2="23.0944" y2="21.1896" width="0.4064" layer="1"/>
+<wire x1="23.0944" y1="21.1896" x2="23.075" y2="21.209" width="0.4064" layer="1"/>
 </signal>
 <signal name="N$28">
 <contactref element="R25" pad="2"/>
 <contactref element="D12" pad="A"/>
-<wire x1="21.717" y1="24.753" x2="22.579" y2="24.753" width="0.4064" layer="1"/>
-<wire x1="22.579" y1="24.753" x2="23.241" y2="24.091" width="0.4064" layer="1"/>
+<wire x1="21.324" y1="22.479" x2="21.324" y2="21.26" width="0.4064" layer="1"/>
+<wire x1="21.324" y1="21.26" x2="21.375" y2="21.209" width="0.4064" layer="1"/>
 </signal>
 <signal name="N$1">

Commit message: WeatherShield_v1
Parts:
- removed LOGO1: OSHW-LOGOM, SparkFun-Aesthetics:OSHW-LOGO-M
- moved R25 3.89 mm to (18.4, 20.4)
- moved D12 2.54 mm to (18.0, 22.5)
- moved C6 2.44 mm to (13.6, 15.7)
- moved C5 1.80 mm to (15.9, 6.48), turned to 90 degrees
Routing:
- net GND: track 12.7 -> 17.1 mm, vias 2 -> 0
- net 3.3V: track 45.8 -> 41.8 mm
- net SDA: track 38.7 -> 34.9 mm
- net 5V: track 4.59 -> 6.86 mm
- net N$5: track 4.27 -> 2.84 mm
- net N$28: track 1.29 -> 2.54 mm
- net SCL: track 43.1 -> 43.8 mm
