File: AirBoard_Shield/WeatherShield_Air.brd (EAGLE design)
At the start: 33 x 26.7 mm, 7 parts, among them U4 MPL3115A2LGA8, U5 HTU21D

Commit message: WeatherShield_v1
Routing:
- net GND: track 17.1 -> 5.10 mm, vias 0 -> 2
Other:
- board text added: "PWR"
Changed lines of the file:
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@@
 <setting verticaltext="up"/>
 </settings>
-<grid distance="5" unitdist="mil" unit="mil" style="lines" multiple="1" display="yes" altdistance="0.005" altunitdist="inch" altunit="inch"/>
+<grid distance="1" unitdist="mil" unit="mil" style="lines" multiple="1" display="yes" altdistance="0.005" altunitdist="inch" altunit="inch"/>
 <layers>
 <layer number="1" name="Top" color="4" fill="1" visible="yes" active="yes"/>
@@
 <layer number="19" name="Unrouted" color="6" fill="1" visible="yes" active="yes"/>
 <layer number="20" name="Dimension" color="15" fill="1" visible="yes" active="yes"/>
-<layer number="21" name="tPlace" color="16" fill="1" visible="yes" active="yes"/>
-<layer number="22" name="bPlace" color="14" fill="1" visible="yes" active="yes"/>
-<layer number="23" name="tOrigins" color="15" fill="1" visible="yes" active="yes"/>
-<layer number="24" name="bOrigins" color="15" fill="1" visible="yes" active="yes"/>
+<layer number="21" name="tPlace" color="16" fill="1" visible="no" active="yes"/>
+<layer number="22" name="bPlace" color="14" fill="1" visible="no" active="yes"/>
+<layer number="23" name="tOrigins" color="15" fill="1" visible="no" active="yes"/>
+<layer number="24" name="bOrigins" color="15" fill="1" visible="no" active="yes"/>
 <layer number="25" name="tNames" color="7" fill="1" visible="no" active="yes"/>
 <layer number="26" name="bNames" color="7" fill="1" visible="no" active="yes"/>
@@
 <layer number="43" name="vRestrict" color="2" fill="10" visible="no" active="yes"/>
 <layer number="44" name="Drills" color="7" fill="1" visible="no" active="yes"/>
-<layer number="45" name="Holes" color="7" fill="1" visible="yes" active="yes"/>
+<layer number="45" name="Holes" color="7" fill="1" visible="no" active="yes"/>
 <layer number="46" name="Milling" color="3" fill="1" visible="no" active="yes"/>
 <layer number="47" name="Measures" color="7" fill="1" visible="no" active="yes"/>
-<layer number="48" name="Document" color="7" fill="1" visible="yes" active="yes"/>
+<layer number="48" name="Document" color="7" fill="1" visible="no" active="yes"/>
 <layer number="49" name="Reference" color="7" fill="1" visible="no" active="yes"/>
 <layer number="50" name="dxf" color="7" fill="1" visible="no" active="yes"/>
-<layer number="51" name="tDocu" color="6" fill="1" visible="yes" active="yes"/>
-<layer number="52" name="bDocu" color="7" fill="1" visible="yes" active="yes"/>
+<layer number="51" name="tDocu" color="6" fill="1" visible="no" active="yes"/>
+<layer number="52" name="bDocu" color="7" fill="1" visible="no" active="yes"/>
 <layer number="53" name="tGND_GNDA" color="7" fill="9" visible="no" active="no"/>
 <layer number="54" name="bGND_GNDA" color="1" fill="9" visible="no" active="no"/>
@@
 <board>
 <plain>
-<text x="11.049" y="1.524" size="1.016" layer="21" ratio="15">FSE Weather Shield V1</text>
+<text x="9.398" y="1.651" size="1.016" layer="1" ratio="15">FSE Weather Shield V1</text>
 <text x="22.86" y="-24.13" size="1.778" layer="27" font="vector" ratio="15">N. Seidle</text>
-<text x="7.239" y="15.621" size="1.27" layer="21" ratio="15" rot="R270">Pressure</text>
-<text x="10.033" y="17.399" size="1.27" layer="21" ratio="15" rot="R90">Humidity</text>
+<text x="8.636" y="14.605" size="1.27" layer="21" ratio="15" rot="R270">Pressure</text>
+<text x="9.779" y="16.002" size="1.27" layer="21" ratio="15" rot="R90">Humidity</text>
 <wire x1="33.274" y1="22.733" x2="33.274" y2="3.683" width="0" layer="20"/>
 <wire x1="0.254" y1="22.733" x2="0.254" y2="3.683" width="0" layer="20"/>
@@
 <circle x="15.24" y="12.319" radius="0.179603125" width="0.4064" layer="1"/>
 <circle x="10.16" y="17.653" radius="0.179603125" width="0.4064" layer="1"/>
+<text x="17.272" y="17.907" size="1.27" layer="21" ratio="15">PWR</text>
 </plain>
 <attributes>
@@
 <contactref element="JP9-DNP2" pad="5"/>
 <contactref element="JP9-DNP2" pad="6"/>
-<wire x1="14.214" y1="18.439" x2="14.224" y2="18.439" width="0.4064" layer="1"/>
-<wire x1="14.224" y1="18.439" x2="14.224" y2="15.9376" width="0.4064" layer="1"/>
-<wire x1="14.224" y1="15.9376" x2="14.4898" y2="15.6718" width="0.4064" layer="1"/>
 <wire x1="23.0944" y1="12.5456" x2="23.0944" y2="12.0454" width="0.4064" layer="1"/>
-<wire x1="23.0944" y1="12.0454" x2="18.415" y2="7.366" width="0.4064" layer="1"/>
-<wire x1="18.415" y1="7.366" x2="15.914" y2="7.366" width="0.4064" layer="1"/>
 <wire x1="15.914" y1="7.366" x2="15.875" y2="7.327" width="0.4064" layer="1"/>
 <wire x1="15.875" y1="7.327" x2="15.875" y2="8.763" width="0.4064" layer="1"/>
 <wire x1="15.875" y1="8.763" x2="15.113" y2="9.525" width="0.4064" layer="1"/>
 <wire x1="15.113" y1="9.525" x2="13.081" y2="9.525" width="0.4064" layer="1"/>
-<wire x1="23.0944" y1="12.0454" x2="25.6344" y2="11.5256" width="0" layer="19" extent="1-1"/>
+<via x="19.05" y="7.62" extent="1-16" drill="0.6"/>
+<via x="19.05" y="5.08" extent="1-16" drill="0.6"/>
+<wire x1="19.05" y1="7.62" x2="19.05" y2="5.08" width="0" layer="19" extent="1-1"/>
 </signal>
 <signal name="3.3V">
@@
 <wire x1="16.637" y1="15.621" x2="15.494" y2="16.764" width="0.4064" layer="1"/>
 <wire x1="15.494" y1="16.764" x2="15.494" y2="18.409" width="0.4064" layer="1"/>
-<wire x1="15.494" y1="18.409" x2="15.464" y2="18.439" width="0.4064" layer="1"/>
 <wire x1="11.714" y1="18.439" x2="11.714" y2="17.429" width="0.4064" layer="1"/>
 <wire x1="11.714" y1="17.429" x2="11.303" y2="17.018" width="0.4064" layer="1"/>
@@
 <wire x1="9.017" y1="7.62" x2="10.541" y2="6.096" width="0.4064" layer="1"/>
 <wire x1="10.541" y1="6.096" x2="13.081" y2="6.096" width="0.4064" layer="1"/>
+<wire x1="15.464" y1="18.439" x2="15.494" y2="18.439" width="0.254" layer="1"/>
+<wire x1="15.494" y1="18.439" x2="15.494" y2="18.409" width="0.254" layer="1"/>
 </signal>
 <signal name="SCL">
