File: Base_Shield/WeatherShield_Base.brd (EAGLE design)
At the start: 58.4 x 67.3 mm, 68 parts, among them Q1 BSS138, Q2 BSS138, U1 DS3231SN, U2 LT3652, U3 TMP100MDBVREP, U4 ADS1015IDGST

Commit message: WeatherShield_v1
Parts:
- renumbered U$1 to SOLAR_CELL, U$6 to BATT
Routing:
- net 5V: track 159.6 -> 158.1 mm, vias 5 -> 4
Changed lines of the file:
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@@
 <layer number="19" name="Unrouted" color="6" fill="1" visible="yes" active="yes"/>
 <layer number="20" name="Dimension" color="15" fill="1" visible="yes" active="yes"/>
-<layer number="21" name="tPlace" color="16" fill="1" visible="yes" active="yes"/>
-<layer number="22" name="bPlace" color="14" fill="1" visible="yes" active="yes"/>
-<layer number="23" name="tOrigins" color="15" fill="1" visible="yes" active="yes"/>
-<layer number="24" name="bOrigins" color="15" fill="1" visible="yes" active="yes"/>
+<layer number="21" name="tPlace" color="16" fill="1" visible="no" active="yes"/>
+<layer number="22" name="bPlace" color="14" fill="1" visible="no" active="yes"/>
+<layer number="23" name="tOrigins" color="15" fill="1" visible="no" active="yes"/>
+<layer number="24" name="bOrigins" color="15" fill="1" visible="no" active="yes"/>
 <layer number="25" name="tNames" color="7" fill="1" visible="no" active="yes"/>
 <layer number="26" name="bNames" color="7" fill="1" visible="no" active="yes"/>
@@
 <layer number="43" name="vRestrict" color="2" fill="10" visible="no" active="yes"/>
 <layer number="44" name="Drills" color="7" fill="1" visible="no" active="yes"/>
-<layer number="45" name="Holes" color="7" fill="1" visible="yes" active="yes"/>
+<layer number="45" name="Holes" color="7" fill="1" visible="no" active="yes"/>
 <layer number="46" name="Milling" color="3" fill="1" visible="no" active="yes"/>
 <layer number="47" name="Measures" color="7" fill="1" visible="no" active="yes"/>
-<layer number="48" name="Document" color="7" fill="1" visible="yes" active="yes"/>
+<layer number="48" name="Document" color="7" fill="1" visible="no" active="yes"/>
 <layer number="49" name="Reference" color="7" fill="1" visible="no" active="yes"/>
 <layer number="50" name="dxf" color="7" fill="1" visible="no" active="yes"/>
-<layer number="51" name="tDocu" color="6" fill="1" visible="yes" active="yes"/>
-<layer number="52" name="bDocu" color="7" fill="1" visible="yes" active="yes"/>
+<layer number="51" name="tDocu" color="6" fill="1" visible="no" active="yes"/>
+<layer number="52" name="bDocu" color="7" fill="1" visible="no" active="yes"/>
 <layer number="53" name="tGND_GNDA" color="7" fill="9" visible="no" active="no"/>
 <layer number="54" name="bGND_GNDA" color="1" fill="9" visible="no" active="no"/>
@@
 <element name="R22" library="pot" package="SM-42/43A" value="" x="17.9832" y="52.7812" rot="R180"/>
 <element name="JP9-DNP1" library="FSEWeatherShield" package="RJ11-STECKER" value="RJ11-BUCHSE" x="11.684" y="0.508"/>
-<element name="U$1" library="FSEWeatherShield" package="XT-60" value="XT-60" x="5.588" y="38.735" rot="R270"/>
-<element name="U$6" library="FSEWeatherShield" package="XT-60" value="XT-60" x="5.588" y="55.372" rot="R270"/>
+<element name="SOLAR_CELL" library="FSEWeatherShield" package="XT-60" value="XT-60" x="5.588" y="38.735" rot="R270"/>
+<element name="BATT" library="FSEWeatherShield" package="XT-60" value="XT-60" x="5.588" y="55.372" rot="R270"/>
 <element name="JP1" library="pinhead" package="1X02" value="" x="47.879" y="17.78" rot="R270"/>
 <element name="JP2" library="pinhead" package="1X02" value="" x="49.657" y="23.622" rot="R270"/>
@@
 <via x="10.5156" y="44.4246" extent="1-16" drill="0.5" diameter="0.254"/>
 <polygon width="0.254" layer="1">
-<vertex x="26.416" y="1.524"/>
+<vertex x="26.289" y="0.254"/>
 <vertex x="26.416" y="28.448"/>
 <vertex x="12.827" y="28.448"/>
-<vertex x="12.827" y="68.834"/>
-<vertex x="1.524" y="68.834"/>
-<vertex x="1.27" y="1.651"/>
+<vertex x="12.446" y="69.088"/>
+<vertex x="1.143" y="69.088"/>
+<vertex x="1.143" y="0.381"/>
 </polygon>
-<contactref element="U$1" pad="NEG"/>
-<contactref element="U$6" pad="NEG"/>
+<contactref element="SOLAR_CELL" pad="NEG"/>
+<contactref element="BATT" pad="NEG"/>
 <contactref element="JP2" pad="2"/>
 <contactref element="JP1" pad="2"/>
@@
 </polygon>
 <contactref element="C5" pad="2"/>
-<via x="51.0286" y="55.8546" extent="1-16" drill="0.5" diameter="0.254"/>
+<via x="51.1556" y="54.8386" extent="1-16" drill="0.5" diameter="0.254"/>
 <contactref element="U4" pad="3"/>
 <contactref element="U4" pad="1"/>
@@
 <wire x1="26.543" y1="64.516" x2="26.543" y2="59.5882" width="0.3048" layer="1"/>
 <wire x1="26.543" y1="59.5882" x2="26.5624" y2="59.5688" width="0.3048" layer="1"/>
-<wire x1="11.8872" y1="24.0284" x2="13.9954" y2="24.0284" width="0.6096" layer="1"/>
-<wire x1="13.9954" y1="24.0284" x2="14.605" y2="24.638" width="0.6096" layer="1"/>
-<wire x1="14.605" y1="24.638" x2="14.605" y2="27.5454" width="0.6096" layer="1"/>
+<wire x1="11.8872" y1="24.0284" x2="13.9954" y2="24.0284" width="0.4064" layer="1"/>
+<wire x1="13.9954" y1="24.0284" x2="14.605" y2="24.638" width="0.4064" layer="1"/>
+<wire x1="14.605" y1="24.638" x2="14.605" y2="27.5454" width="0.4064" layer="1"/>
 <wire x1="14.605" y1="27.5454" x2="14.566" y2="27.5844" width="0.6096" layer="1"/>
-<wire x1="11.8872" y1="24.0284" x2="10.3006" y2="24.0284" width="0.6096" layer="1"/>
-<wire x1="10.3006" y1="24.0284" x2="9.525" y2="24.804" width="0.6096" layer="1"/>
+<wire x1="11.8872" y1="24.0284" x2="10.3006" y2="24.0284" width="0.4064" layer="1"/>
+<wire x1="10.3006" y1="24.0284" x2="9.525" y2="24.804" width="0.4064" layer="1"/>
 <wire x1="19.314" y1="8.808" x2="19.314" y2="6.487" width="0.4064" layer="1"/>
 <wire x1="19.314" y1="6.487" x2="18.415" y2="5.588" width="0.4064" layer="1"/>
@@
 <wire x1="41.275" y1="47.625" x2="42.037" y2="46.863" width="0.3048" layer="1"/>
 <via x="42.037" y="46.863" extent="1-16" drill="0.6"/>
-<wire x1="42.037" y1="46.863" x2="42.037" y2="45.339" width="0.3048" layer="16"/>
-<wire x1="42.037" y1="45.339" x2="43.053" y2="44.323" width="0.3048" layer="16"/>
-<via x="43.053" y="44.323" extent="1-16" drill="0.6"/>
-<wire x1="43.053" y1="44.323" x2="44.45" y2="44.323" width="0.3048" layer="1"/>
+<wire x1="42.037" y1="46.863" x2="42.037" y2="45.085" width="0.3048" layer="16"/>
+<via x="43.307" y="44.323" extent="1-16" drill="0.6"/>
+<wire x1="43.307" y1="44.323" x2="44.45" y2="44.323" width="0.3048" layer="1"/>
+<wire x1="42.037" y1="45.085" x2="42.799" y2="44.323" width="0.3048" layer="16"/>
+<wire x1="42.799" y1="44.323" x2="43.307" y2="44.323" width="0.3048" layer="16"/>
 </signal>
 <signal name="5V">
@@
 <wire x1="40.513" y1="41.656" x2="40.513" y2="41.568" width="0.4064" layer="1"/>
 <wire x1="40.513" y1="41.568" x2="38.989" y2="41.568" width="0.4064" layer="1"/>
-<wire x1="44.45" y1="41.568" x2="43.395" y2="41.568" width="0.4064" layer="1"/>
-<wire x1="43.395" y1="41.568" x2="43.18" y2="41.783" width="0.4064" layer="1"/>
-<via x="43.18" y="41.783" extent="1-16" drill="0.6"/>
-<wire x1="43.18" y1="41.783" x2="43.18" y2="35.687" width="0.4064" layer="16"/>
 <wire x1="43.18" y1="35.687" x2="46.482" y2="32.385" width="0.4064" layer="16"/>
 <wire x1="46.482" y1="32.385" x2="48.895" y2="32.385" width="0.4064" layer="16"/>
@@
 <wire x1="50.4444" y1="30.4546" x2="50.927" y2="29.972" width="0.4064" layer="1"/>
 <wire x1="50.927" y1="29.972" x2="50.927" y2="29.464" width="0.4064" layer="1"/>
+<wire x1="43.18" y1="35.687" x2="43.18" y2="41.656" width="0.4064" layer="16"/>
 <wire x1="56.183" y1="58.686" x2="56.183" y2="56.146" width="0" layer="19" extent="1-1"/>
 </signal>
@@
 <contactref element="JP10-DNP" pad="2"/>
 <wire x1="41.6714" y1="62.1088" x2="41.5502" y2="62.23" width="0.3048" layer="1"/>
-<wire x1="41.5502" y1="62.23" x2="33.147" y2="62.23" width="0.3048" layer="1"/>
+<wire x1="41.5502" y1="62.23" x2="33.909" y2="62.23" width="0.3048" layer="1"/>
 <wire x1="29.1846" y1="51.562" x2="30.353" y2="51.562" width="0.3048" layer="1"/>
 <wire x1="30.353" y1="51.562" x2="30.607" y2="51.816" width="0.3048" layer="1"/>
 <wire x1="30.607" y1="51.816" x2="30.607" y2="54.356" width="0.3048" layer="1"/>
-<wire x1="33.147" y1="62.23" x2="31.281" y2="60.364" width="0.3048" layer="1"/>
-<wire x1="31.281" y1="60.364" x2="31.281" y2="55.499" width="0.3048" layer="1"/>
 <wire x1="30.607" y1="54.356" x2="31.281" y2="55.03" width="0.3048" layer="1"/>
 <wire x1="31.281" y1="55.03" x2="31.281" y2="55.499" width="0.3048" layer="1"/>
+<wire x1="31.281" y1="55.499" x2="31.369" y2="55.499" width="0.3048" layer="1"/>
+<wire x1="31.369" y1="55.499" x2="31.369" y2="59.69" width="0.3048" layer="1"/>
+<wire x1="31.369" y1="59.69" x2="33.909" y2="62.23" width="0.3048" layer="1"/>
 </signal>
 <signal name="N$6">
@@
 <wire x1="19.5066" y1="48.5896" x2="19.6082" y2="48.5896" width="0.4064" layer="1"/>
 <wire x1="19.6082" y1="48.5896" x2="20.2946" y2="49.276" width="0.4064" layer="1"/>
-<contactref element="U$1" pad="POS"/>
+<contactref element="SOLAR_CELL" pad="POS"/>
 <wire x1="15.265" y1="54.229" x2="14.478" y2="54.229" width="0.6096" layer="1"/>
 <wire x1="14.478" y1="54.229" x2="10.541" y2="50.292" width="0.6096" layer="1"/>
@@
 <wire x1="12.319" y1="57.912" x2="12.319" y2="58.332" width="0.6096" layer="1"/>
 <wire x1="12.319" y1="58.332" x2="13.589" y2="59.602" width="0.6096" layer="1"/>
-<contactref element="U$6" pad="POS"/>
-<wire x1="11.7602" y1="33.528" x2="9.017" y2="36.2712" width="0.6096" layer="1"/>
-<wire x1="9.017" y1="36.2712" x2="9.017" y2="42.037" width="0.6096" layer="1"/>
-<wire x1="9.017" y1="42.037" x2="8.255" y2="42.799" width="0.6096" layer="1"/>
+<contactref element="BATT" pad="POS"/>
+<wire x1="9.271" y1="41.783" x2="8.255" y2="42.799" width="0.6096" layer="1"/>
 <wire x1="11.938" y1="47.879" x2="8.255" y2="44.196" width="0.6096" layer="16"/>
 <wire x1="8.255" y1="44.196" x2="8.255" y2="42.799" width="0.6096" layer="16"/>
@@
 <wire x1="42.545" y1="28.702" x2="42.545" y2="27.175" width="0.6096" layer="1"/>
 <wire x1="42.545" y1="27.175" x2="42.5226" y2="27.1526" width="0.6096" layer="1"/>
+<wire x1="9.271" y1="41.783" x2="9.271" y2="36.0172" width="0.6096" layer="1"/>
+<wire x1="9.271" y1="36.0172" x2="11.7602" y2="33.528" width="0.6096" layer="1"/>
 </signal>
 <signal name="N$15">

Commit message: WeatherShield_v1
Parts:
- removed G1: 3V, battery:CELL_RETAINER_11.6MM
- removed JP6: (no value), pinhead:1X01
- added JP10, JP11, JP12, JP9: (no value), pinhead:1X01
- added R11, R13: 0, rcl:R0603
- added TP2: SET, testpad:B1,27
- added U$1: BATTERIE_HALTER_CR1225, FSEWeatherShield:BATTERIE_HALTER_CR1225
- moved R10 4.75 mm to (12.1, 35.9)
- moved JP3 3.54 mm to (12.4, 31.4)
- moved R5 1.83 mm to (46.0, 43.4)
- moved D1 1.78 mm to (13.6, 65.0)
- moved D3 1.78 mm to (16.3, 65.0)
- moved R9 1.70 mm to (11.7, 38.8), turned to 0 degrees
- moved R4 1.69 mm to (38.6, 44.1), turned to 180 degrees
- moved C5 1.42 mm to (43.3, 34.7)
- moved U3 1.42 mm to (39.5, 34.7)
- moved R20 1.30 mm to (13.4, 44.3)
- moved R7 1.27 mm to (46.0, 7.37)
- moved C10 0.80 mm to (19.1, 39.7)
- moved D2 0.63 mm to (44.7, 5.08), turned to 180 degrees
Connections:
- removed net N$14: JP6.1, U4.5
- removed net N$6: G1.P+@1, G1.P+@2, U1.14
- new net FAULT_PIN: D1.A, PCB1.7, R1.2
- new net N$1: R13.1, R9.2
- new net N$2: R10.2, R11.1
- new net RTC_BATT: U$1.P, U1.14, U4.5
- net FB: now also R13.2; no longer R9.2
- net GND: now also U$1.N; no longer G1.N-
- net HV_SCL: now also JP9.1
- net HV_SDA: now also JP12.1
- net N$16: now also R11.2; no longer R10.2
- net N$3: now also PCB1.16; no longer D1.A, R1.2
- net SCL: now also JP11.1
- net SDA: now also JP10.1
- net V_BATT: now also TP2.TP
Routing:
- net RTC_BATT: track 0.00 -> 62.2 mm, vias 0 -> 2
- net FAULT_PIN: track 0.00 -> 52.9 mm, vias 0 -> 1
- net N$6: track 37.6 -> 0.00 mm, vias 1 -> 0
- net 3.3V: track 187.9 -> 170.4 mm
- net HV_SCL: track 21.5 -> 35.0 mm, vias 2 -> 4
- net SCL: track 73.9 -> 84.4 mm
- net GND: track 30.4 -> 23.2 mm, vias 9 -> 8
- net HV_SDA: track 13.6 -> 20.5 mm
- net FB: track 3.18 -> 9.95 mm
- net RAIN: track 50.7 -> 56.7 mm, vias 1 -> 0
- net SDA: track 77.6 -> 83.0 mm
- net N$16: track 27.1 -> 31.7 mm
- net N$14: track 4.46 -> 0.00 mm
- net N$2: track 0.00 -> 2.35 mm
- net N$1: track 0.00 -> 1.92 mm
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Other:
- board text added: "User LED"
- board text removed: "Pwr"

Commit message: WeatherShield_v1
Parts:
- moved C1 11.2 mm to (6.96, 18.7), turned to 270 degrees
- moved C8 2.96 mm to (8.00, 23.1), turned to 270 degrees
Routing:
- net 3.3V: track 170.4 -> 163.6 mm, vias 3 -> 4
- net !CHRG: track 23.5 -> 21.7 mm
- net FAULT_PIN: track 52.9 -> 51.9 mm
Other:
- board text added: "AirBoard"
- board text added: "FSE Weather Shield V1 (2016)"
- board text removed: "FSE Weather Shield V1"

Commit message: WeatherShield_v1
Parts:
- R10: value 24k -> 68k
- R9: value 9.1k -> 22k
- RTCBAT: value BATTERIE_HALTER_CR1225 -> CR1225
- moved TP2 4.58 mm to (14.9, 57.1)
- moved D2 1.65 mm to (46.4, 5.08)
- moved R7 1.42 mm to (47.4, 7.11)
- renumbered U$1 to RTCBAT
Routing:
- net STAT3: track 13.7 -> 11.6 mm
- net V_BATT: track 78.5 -> 76.7 mm
- net 3.3V: track 163.6 -> 164.5 mm
- net GND: vias 8 -> 9
Other:
- board text added: "FSE Weather Shield V1"
- board text added: "UserLED"
- board text removed: "FSE Weather Shield V1 (2016)"
- board text removed: "User LED"

Commit message: WeatherShield_v1
Parts:
- removed D1: Red, SparkFun:LED-0603
- removed D3: Green, SparkFun:LED-0603
- removed R22: (no value), pot:SM-42/43A
- added U$1: POT10K, FSEWeatherShield:POT_TS63Y_10K
- added U$2: HSMF_C158, FSEWeatherShield:HSNF_C158
- moved TP1 9.33 mm to (13.4, 51.7)
- moved TP2 6.33 mm to (9.91, 61.1)
- moved R1 5.77 mm to (19.3, 61.2)
- moved R6 1.59 mm to (17.7, 61.2)
- moved SOLAR_CELL 1.53 mm to (5.71, 37.2)
Connections:
- net !CHRG: now also U$2.C1; no longer D3.C
- net !FAULT: now also U$2.C2; no longer D1.C
- net 3.3V: now also R1.1, R6.1
- net FAULT_PIN: now also U$2.A2; no longer D1.A
- net GND: now also U$1.1; no longer R22.1
- net N$7: now also U$2.A1; no longer D3.A
- net SET: now also U$1.2; no longer R22.2
- net VIN: now also U$1.3; no longer R22.3
- net V_BATT: no longer R1.1, R6.1
Routing:
- net GND: track 23.2 -> 8.51 mm
- net 3.3V: track 164.5 -> 175.8 mm
- net VIN: track 36.1 -> 43.8 mm, vias 0 -> 1
- net V_BATT: track 76.7 -> 71.8 mm, vias 3 -> 1
- net SET: track 8.01 -> 11.0 mm
- net !CHRG: track 21.7 -> 19.2 mm
- net FAULT_PIN: track 51.9 -> 50.7 mm
- net !FAULT: track 22.5 -> 23.4 mm

Commit message: WeatherShield_v1
Parts:
- removed U$2: HSMF_C158, FSEWeatherShield:HSNF_C158
- added U$3: VLMV3100, FSEWeatherShield:VLMV3100
- R1, R6: value 1K -> >=290
- moved R6 4.58 mm to (13.1, 61.5), turned to 270 degrees
- moved R1 2.90 mm to (17.0, 59.4), turned to 270 degrees
Connections:
- removed net N$7: R6.2, U$2.A1
- new net N$4: R6.1, U$3.A_GREEN
- net !CHRG: now also R6.2; no longer U$2.C1
- net !FAULT: now also R1.2; no longer U$2.C2
- net 3.3V: no longer R1.1, R6.1
- net 5V: now also U$3.C
- net FAULT_PIN: now also R1.1, U$3.A_RED; no longer R1.2, U$2.A2
Routing:
- net 5V: track 158.4 -> 203.4 mm
- net 3.3V: track 175.8 -> 167.8 mm
- net !FAULT: track 23.4 -> 16.5 mm
- net FAULT_PIN: track 50.7 -> 45.1 mm
- net N$7: track 3.18 -> 0.00 mm
- net N$4: track 0.00 -> 2.14 mm
- net !CHRG: track 19.2 -> 17.8 mm, vias 2 -> 0
- net HV_SCL: track 35.0 -> 34.1 mm

Commit message: WeatherShield_v1
Routing:
- net 3.3V: track 167.8 -> 172.0 mm, vias 4 -> 5
- net HV_SCL: track 34.1 -> 37.1 mm
- net RAIN: track 56.7 -> 58.4 mm
- net 5V: track 203.4 -> 202.2 mm
- net GND: vias 9 -> 10

Commit message: WeatherShield_v1
Parts:
- removed U$3: VLMV3100, FSEWeatherShield:VLMV3100
- added LED_GREEN, LED_RED: (no value), led:SML0603
- moved PCB1 65.7 mm to (0.00, 2.67), turned to 0 degrees
- moved JP9-DNP1 57.6 mm to (67.8, 13.2), turned to 90 degrees
- moved JP10-DNP 55.0 mm to (-2.08, 50.8), turned to 270 degrees
- moved JP9-DNP 50.2 mm to (-2.08, 34.7), turned to 270 degrees
- moved TP2 49.7 mm to (7.24, 11.4), turned to 90 degrees
- moved BATT 48.8 mm to (13.0, 7.11), turned to 0 degrees
- moved R6 47.3 mm to (6.86, 14.6), turned to 0 degrees
- moved D2 46.0 mm to (63.2, 47.9), turned to 270 degrees
- moved R7 44.0 mm to (61.2, 48.9), turned to 270 degrees
- moved C1 43.9 mm to (49.7, 8.48), turned to 0 degrees
- moved R1 41.7 mm to (8.89, 18.5), turned to 0 degrees
- moved C8 39.6 mm to (45.2, 9.53), turned to 0 degrees
- moved C14 39.5 mm to (59.2, 45.7), turned to 90 degrees
- moved C15 39.5 mm to (60.2, 42.6), turned to 270 degrees
- moved SOLAR_CELL 39.3 mm to (31.1, 7.24), turned to 0 degrees
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Connections:
- net 5V: now also LED_GREEN.A, LED_RED.A; no longer U$3.C
- net FAULT_PIN: now also LED_RED.C; no longer U$3.A_RED
- net N$4: now also LED_GREEN.C; no longer U$3.A_GREEN
Routing:
- net 5V: track 202.2 -> 204.2 mm
- net FAULT_PIN: track 45.1 -> 46.2 mm
Other:
- board size 58.4 x 67.3 mm -> 67.3 x 58.4 mm
