File: 01_EagleDocuments/Base_Shield/WeatherShield_Base.sch (EAGLE design)
At the start: 74 parts, among them Q1 BSS138, Q2 BSS138, U1 DS3231SN, U2 LT3652, U3 TMP100MDBVREP, U4 ADS1015IDGST

Commit message: WeatherShield_v1
Parts:
- R17: value 10k -> 20k
Connections:
- net 3.3V: now also R17.1
- net 5V: no longer R17.1
Changed lines of the file:
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@@
 <?xml version="1.0" encoding="utf-8"?>
 <!DOCTYPE eagle SYSTEM "eagle.dtd">
-<eagle version="7.3.0">
+<eagle version="7.4.0">
 <drawing>
 <settings>
@@
 <part name="JP9-DNP" library="FSEWeatherShield" deviceset="RJ11-BUCHSE" device="" value="RJ11-RAIN"/>
 <part name="GND15" library="SparkFun" deviceset="GND" device=""/>
-<part name="R17" library="rcl" deviceset="R-EU_" device="R0603" value="10k"/>
+<part name="R17" library="rcl" deviceset="R-EU_" device="R0603" value="20k"/>
 <part name="R14" library="rcl" deviceset="R-EU_" device="R0603" value="3k9"/>
 <part name="GND21" library="SparkFun" deviceset="GND" device=""/>
-<part name="SUPPLY7" library="SparkFun-Aesthetics" deviceset="5V" device=""/>
 <part name="U1" library="FSE_Weather_Shield" deviceset="DS3231SN" device=""/>
 <part name="GND1" library="SparkFun" deviceset="GND" device=""/>
@@
 <part name="LED_RED" library="led" deviceset="LED" device="SML0603"/>
 <part name="LED_GREEN" library="led" deviceset="LED" device="SML0603"/>
+<part name="P+7" library="SparkFun" deviceset="3.3V" device=""/>
 </parts>
 <sheets>
@@
 </instance>
 <instance part="GND21" gate="1" x="22.86" y="73.66" rot="MR0"/>
-<instance part="SUPPLY7" gate="G$1" x="27.94" y="106.68"/>
 <instance part="U1" gate="A" x="142.24" y="76.2"/>
 <instance part="GND1" gate="1" x="129.54" y="60.96" rot="MR0"/>
@@
 <instance part="LED_RED" gate="G$1" x="205.74" y="162.56" rot="R90"/>
 <instance part="LED_GREEN" gate="G$1" x="205.74" y="157.48" rot="R90"/>
+<instance part="P+7" gate="G$1" x="27.94" y="106.68"/>
 </instances>
 <busses>
@@
 <pinref part="P+13" gate="G$1" pin="3.3V"/>
 </segment>
+<segment>
+<pinref part="R17" gate="G$1" pin="1"/>
+<pinref part="P+7" gate="G$1" pin="3.3V"/>
+</segment>
 </net>
 <net name="SCL" class="0">
@@
 </segment>
 <segment>
-<pinref part="R17" gate="G$1" pin="1"/>
-<pinref part="SUPPLY7" gate="G$1" pin="5V"/>
-</segment>
-<segment>

Commit message: WeatherShield_v1
Connections:
- new net N$5: U3.AD0
- net GND: no longer U3.AD0
Changed lines of the file:
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@@
 <instance part="JP5" gate="A" x="175.26" y="81.28" rot="R180"/>
 <instance part="U3" gate="A" x="27.94" y="55.88"/>
-<instance part="GND12" gate="1" x="7.62" y="48.26" rot="MR0"/>
+<instance part="GND12" gate="1" x="5.08" y="48.26" rot="MR0"/>
 <instance part="P+4" gate="G$1" x="7.62" y="66.04"/>
 <instance part="C5" gate="G$1" x="2.54" y="60.96"/>
@@
 <segment>
 <pinref part="U3" gate="A" pin="GND"/>
-<wire x1="10.16" y1="58.42" x2="7.62" y2="58.42" width="0.1524" layer="91"/>
-<wire x1="7.62" y1="58.42" x2="7.62" y2="50.8" width="0.1524" layer="91"/>
+<wire x1="10.16" y1="58.42" x2="5.08" y2="58.42" width="0.1524" layer="91"/>
+<wire x1="5.08" y1="58.42" x2="5.08" y2="50.8" width="0.1524" layer="91"/>
 <pinref part="GND12" gate="1" pin="GND"/>
-<pinref part="U3" gate="A" pin="AD0"/>
-<wire x1="10.16" y1="55.88" x2="7.62" y2="50.8" width="0.1524" layer="91"/>
-<pinref part="U3" gate="A" pin="AD1"/>
-<wire x1="35.56" y1="55.88" x2="35.56" y2="50.8" width="0.1524" layer="91"/>
-<wire x1="35.56" y1="50.8" x2="7.62" y2="50.8" width="0.1524" layer="91"/>
-<junction x="7.62" y="50.8"/>
-<junction x="7.62" y="50.8"/>
+<wire x1="40.64" y1="50.8" x2="5.08" y2="50.8" width="0.1524" layer="91"/>
+<junction x="5.08" y="50.8"/>
+<junction x="5.08" y="50.8"/>
 <pinref part="C5" gate="G$1" pin="2"/>
 <wire x1="2.54" y1="55.88" x2="2.54" y2="50.8" width="0.1524" layer="91"/>
-<wire x1="2.54" y1="50.8" x2="7.62" y2="50.8" width="0.1524" layer="91"/>
+<wire x1="2.54" y1="50.8" x2="5.08" y2="50.8" width="0.1524" layer="91"/>
+<pinref part="U3" gate="A" pin="AD1"/>
+<wire x1="35.56" y1="55.88" x2="40.64" y2="55.88" width="0.1524" layer="91"/>
+<wire x1="40.64" y1="50.8" x2="40.64" y2="55.88" width="0.1524" layer="91"/>
 </segment>
 <segment>
@@
 </segment>
 </net>
+<net name="N$5" class="0">
+<segment>
+<pinref part="U3" gate="A" pin="AD0"/>
+<wire x1="10.16" y1="55.88" x2="7.62" y2="55.88" width="0.1524" layer="91"/>
+</segment>
+</net>
